File: hw/morse-tx/elec/layout/default/morse-tx.kicad_pcb (KiCad board)
At the start: 2 copper layers, 225.7 x 100.8 mm, 0 parts

Commit message: Partial commit
Parts:
- added C1: Multilayer Ceramic Capacitors MLCC - SMD/SMT 1uF 50V 0603 R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, lib:C0603, F.Cu at (115.3, 84.8)
- added C2: Multilayer Ceramic Capacitors MLCC - SMD/SMT 1uF 50V 0603 R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, lib:C0603, F.Cu at (117.1, 84.8)
- added C3: Multilayer Ceramic Capacitors MLCC - SMD/SMT 2.2uF 10V 0603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, lib:C0603, F.Cu at (129.8, 84.8)
- added C4: , lib:C0805, F.Cu at (127.8, 85.0)
- added C5: Multilayer Ceramic Capacitors MLCC - SMD/SMT 1uF 50V 0603 R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, lib:C0603, F.Cu at (112.8, 84.8)
- added C6: Multilayer Ceramic Capacitors MLCC - SMD/SMT 1uF 50V 0603 R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, lib:C0603, F.Cu at (111.0, 84.8)
- added R1: Chip Resistor - Surface Mount 560KOhms ±5% 1/10W 0603 RoHS, lib:R0603, F.Cu at (125.7, 84.8)
- added R2: Chip Resistor - Surface Mount 4.7KOhms ±5% 1/10W 0603 RoHS, lib:R0603, F.Cu at (121.0, 85.9)
- added R3: Chip Resistor - Surface Mount 4.7KOhms ±5% 1/10W 0603 RoHS, lib:R0603, F.Cu at (121.9, 84.1)
- added U1: , lib:SOT-23-5_L3.0-W1.7-P0.95-LS2.8-BR, F.Cu at (128.3, 100.7)
- added U2: , lib:IND-SMD_L5.4-W5.2_FXL0530, F.Cu at (117.7, 103.8)
- added U3: , lib:OLED_0.96-30P-P0.70-12864, F.Cu at (120.3, 81.3)
- added U4: , Connector:Tag-Connect_TC2050-IDC-NL_2x05_P1.27mm_Vertical, F.Cu at (139.7, 99.7)
- added U5: , lib:TSSOP-28_L9.7-W4.4-P0.65-LS6.4-BL, F.Cu at (140.6, 111.4)
Other:
- board outline removed
